File: jmny-crkt/power.kicad_sch (KiCad schematic)
At the start: 0 parts

Commit message: Made some progress on the BQ25505 in the old schematic. Will polish it off and import into new project next.
Parts:
- added C1, C4: 10uF, Capacitor_SMD:C_0805_2012Metric, symbol Device:C
- added C2, C3, C5: 10nF, Capacitor_SMD:C_0402_1005Metric, symbol Device:C
- added L1: 22uH, Inductor_SMD:L_0805_2012Metric, symbol Device:L
- added R1, R2: 5.11 MR, Resistor_SMD:R_0402_1005Metric, symbol Device:R
- added R3: 6.2 MR, Resistor_SMD:R_0402_1005Metric, symbol Device:R
- added R4: 7.5 MR, Resistor_SMD:R_0402_1005Metric, symbol Device:R
- added R5: 1.5 MR, Resistor_SMD:R_0402_1005Metric, symbol Device:R
- added R6: 6.8 MR, Resistor_SMD:R_0402_1005Metric, symbol Device:R
- added R7: 5.1 MR, Resistor_SMD:R_0402_1005Metric, symbol Device:R
- added U1, U2: 4700uF, footprint:CAP-TH_BD10.0-F5.00-D0.6-FD, symbol HS0J478M1016PC:HS0J478M1016PC
- added U3: BQ25505RGRT, BQ25505RGRT:BQ25505RGRT, symbol BQ25505RGRT:BQ25505RGRT
Connections:
- new net: C1.1, L1.1, R1.1, U3.2 (VIN_DC)
- new net: L1.2, U3.20 (LBOOST)
- new net: R1.2, R2.1, U3.3 (VOC_SAMP)
- new net: C2.1, U3.4 (VREF_SAMP)
- new net BAT_OV: R3.2, R4.1, U3.7 (VBAT_OV)
- new net GND: C1.2, C2.2, C3.2, C4.2, C5.2, R2.2, R4.2, R7.2, U1.2, U2.2, U3.1 (VSS-1), U3.15 (VSS), U3.21 (E_PAD)
- new net OK_HYST: R5.2, R6.1, U3.11 (OK_HYST)
- new net OK_PROG: R6.2, R7.1, U3.12 (OK_PROG)
- new net VBAT_PRI: U3.14 (VBAT_PRI)
- new net VCAP: C3.1, U1.1, U2.1, U3.18 (VBAT_SEC)
- new net V_RDIV: R3.1, R5.1, U3.8 (VRDIV)
- new net Vstore: C4.1, C5.1, U3.19 (VSTOR)
- new net ~{EN}: U3.5 (~{EN})
- no-connect marks 0 -> 1
