File: crktboi/oscillator.kicad_sch (KiCad schematic)
At the start: 10 parts, among them Q1 BC847, Q2 BC847, Q3 2N7002, U1 GSC1102YB-3V4000

Commit message: Added a plan document & updated  design with tweaks for 3S3P photodiodes
Changed lines of the file:
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@@
-		)
-	)
-	(hierarchical_label "VBAT_OK"
-		(shape input)
-		(at 27.94 62.23 180)
-		(effects
-			(font
-				(size 1.27 1.27)
-			)
-			(justify right)
 		)
 	)

Commit message: Added LCSC part numbers to each part in the schematic
Parts:
- C1, C2: LCSC (none) -> C100040
- Q1, Q2: LCSC (none) -> C2138
- Q3: LCSC (none) -> C8545
- R1, R4: LCSC (none) -> C22548
- R2, R3: LCSC (none) -> C22890
Changed lines of the file:
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@@
 			)
 		)
-		(property "LCSC" ""
+		(property "LCSC" "C22890"
 			(at 109.22 68.58 0)
 			(hide yes)
@@
 			)
 		)
-		(property "LCSC" ""
+		(property "LCSC" "C100040"
 			(at 116.84 81.28 90)
 			(hide yes)
@@
 			)
 		)
-		(property "LCSC" ""
+		(property "LCSC" "C2138"
 			(at 121.92 96.52 0)
 			(hide yes)
@@
 			)
 		)
-		(property "LCSC" ""
+		(property "LCSC" "C2138"
 			(at 78.74 96.52 0)
 			(hide yes)
@@
 			)
 		)
-		(property "LCSC" ""
+		(property "LCSC" "C8545"
 			(at 146.05 87.63 0)
 			(hide yes)
@@
 			)
 		)
-		(property "LCSC" ""
+		(property "LCSC" "C22890"
 			(at 90.17 68.58 0)
 			(hide yes)
@@
 			)
 		)
-		(property "LCSC" ""
+		(property "LCSC" "C22548"
 			(at 76.2 68.58 0)
 			(hide yes)
@@
 			)
 		)
-		(property "LCSC" ""
+		(property "LCSC" "C100040"
 			(at 82.55 81.28 90)
 			(hide yes)
@@
 			)
 		)
-		(property "LCSC" ""
+		(property "LCSC" "C22548"
 			(at 124.46 68.58 0)
 			(hide yes)
