File: crktboi/crktboi.kicad_pcb (KiCad board)
At the start: 2 copper layers, 66 x 21.5 mm, 38 parts, among them Q1 BC847, Q2 BC847, Q3 2N7002, Q4 2N7002, Q5 AO3401A, U1 GSC1102YB-3V4000, U2 VBPW34S, U3 VBPW34S, U4 BQ25505RGRT

Commit message: Added BAT54J diodes to the input connectors of the PV headers
Parts:
- added D2: BAT54J, Diode_SMD:D_SOD-323F, F.Cu at (136.9, 106.2)
- added D3: BAT54J, Diode_SMD:D_SOD-323F, F.Cu at (136.9, 93.9)
- moved R11 2.00 mm to (136.4, 97.3)
- moved C6 1.27 mm to (138.9, 106.2)
Connections:
- TP1 pad 1: Net-(D1-K) -> Net-(D3-A)
- TP2 pad 1: Net-(D1-K) -> Net-(D2-A)
Routing:
- net Net-(D3-A): track 0.00 -> 6.37 mm
- net Net-(D2-A): track 0.00 -> 5.76 mm
- net Net-(D1-K): track 41.1 -> 39.3 mm, vias 1 -> 3

Commit message: Added a graphic to the back of the base board of a Cicada
Parts:
- added G***: LOGO, LOGO, B.Cu at (148.8, 99.9)

Commit message: removed the cicada graphic a it was too busy
Parts:
- removed G***: LOGO, LOGO

Commit message: Updated Gerbers of new body PCB
Routing:
- net GND: vias 26 -> 29
Changed lines of the file:
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@@
+	)
+	(via
+		(at 137.5 106.5)
+		(size 0.6)
+		(drill 0.3)
+		(layers "F.Cu" "B.Cu")
+		(free yes)
+		(net "GND")
 	)
 	(via
@@
 	)
 	(via
+		(at 136.25 96)
+		(size 0.6)
+		(drill 0.3)
+		(layers "F.Cu" "B.Cu")
+		(free yes)
+		(net "GND")
+	)
+	(via
 		(at 130.1 100)
 		(size 0.5)
@@
 	)
 	(via
+		(at 140 108.5)
+		(size 0.6)
+		(drill 0.3)
+		(layers "F.Cu" "B.Cu")
+		(free yes)
+		(net "GND")
+	)
+	(via
 		(at 124.1 95.3)
 		(size 0.5)
@@
 	)
 	(segment
+		(start 133.3064 92.0536)
+		(end 136.153599 92.0536)
+		(width 0.3)
+		(layer "F.Cu")
+		(net "Net-(D3-A)")
+	)
+	(segment
+		(start 136.153599 92.0536)
+		(end 136.9 92.800001)
+		(width 0.3)
+		(layer "F.Cu")
+		(net "Net-(D3-A)")
+	)
+	(segment
+		(start 131.56 93.8)
+		(end 133.3064 92.0536)
+		(width 0.3)
+		(layer "F.Cu")
+		(net "Net-(D3-A)")
+	)
+	(segment
 		(start 138.46 103.16)
 		(end 138.13 102.83)
@@
 	)
 	(segment
+		(start 136.859999 107.34)
+		(end 132.77 107.34)
+		(width 0.3)
+		(layer "F.Cu")
+		(net "Net-(D2-A)")
+	)
+	(segment
+		(start 136.9 107.299999)
+		(end 136.859999 107.34)
+		(width 0.3)
+		(layer "F.Cu")
+		(net "Net-(D2-A)")
+	)
+	(segment
+		(start 132.77 107.34)
+		(end 131.63 106.2)
+		(width 0.3)
+		(layer "F.Cu")
+		(net "Net-(D2-A)")
+	)
+	(segment
 		(start 141.88 99.509999)
 		(end 141 99.509999)
@@
 		(net "Net-(Q2-C)")
 	)
-	(segment
-		(start 136.859999 107.34)
-		(end 132.77 107.34)
-		(width 0.3)
-		(layer "F.Cu")
-		(net "Net-(D2-A)")
-	)
-	(segment
-		(start 136.9 107.299999)
-		(end 136.859999 107.34)
-		(width 0.3)
-		(layer "F.Cu")
-		(net "Net-(D2-A)")
-	)
-	(segment
-		(start 132.77 107.34)
-		(end 131.63 106.2)
-		(width 0.3)
-		(layer "F.Cu")
-		(net "Net-(D2-A)")
-	)
-	(segment
-		(start 133.3064 92.0536)
-		(end 136.153599 92.0536)
-		(width 0.3)
-		(layer "F.Cu")
-		(net "Net-(D3-A)")
-	)
-	(segment
-		(start 136.153599 92.0536)
-		(end 136.9 92.800001)
-		(width 0.3)
-		(layer "F.Cu")
-		(net "Net-(D3-A)")
-	)
-	(segment
-		(start 131.56 93.8)
-		(end 133.3064 92.0536)
-		(width 0.3)
-		(layer "F.Cu")
-		(net "Net-(D3-A)")
-	)
 	(zone
